File: SwiftLeeds.kicad_sch (KiCad schematic)
At the start: 11 parts

Commit message: V.... 5 I think? Idk anymore, time has become one long unending torture
Parts:
- D1, D2, D3, D4, D5: footprint LED_SMD:LED_0805_2012Metric -> LED_SMD:LED_0805_Side
Changed lines of the file:
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@@
       (effects (font (size 1.27 1.27)) (justify right))
     )
-    (property "Footprint" "LED_SMD:LED_0805_2012Metric" (id 2) (at 151.13 97.79 0)
+    (property "Footprint" "LED_SMD:LED_0805_Side" (id 2) (at 151.13 97.79 0)
       (effects (font (size 1.27 1.27)) hide)
     )
@@
       (effects (font (size 1.27 1.27)) (justify right))
     )
-    (property "Footprint" "LED_SMD:LED_0805_2012Metric" (id 2) (at 144.78 97.79 0)
+    (property "Footprint" "LED_SMD:LED_0805_Side" (id 2) (at 144.78 97.79 0)
       (effects (font (size 1.27 1.27)) hide)
     )
@@
       (effects (font (size 1.27 1.27)) (justify right))
     )
-    (property "Footprint" "LED_SMD:LED_0805_2012Metric" (id 2) (at 163.83 97.79 0)
+    (property "Footprint" "LED_SMD:LED_0805_Side" (id 2) (at 163.83 97.79 0)
       (effects (font (size 1.27 1.27)) hide)
     )
@@
       (effects (font (size 1.27 1.27)) (justify right))
     )
-    (property "Footprint" "LED_SMD:LED_0805_2012Metric" (id 2) (at 139.7 97.79 0)
+    (property "Footprint" "LED_SMD:LED_0805_Side" (id 2) (at 139.7 97.79 0)
       (effects (font (size 1.27 1.27)) hide)
     )
@@
       (effects (font (size 1.27 1.27)) (justify right))
     )
-    (property "Footprint" "LED_SMD:LED_0805_2012Metric" (id 2) (at 156.21 97.79 0)
+    (property "Footprint" "LED_SMD:LED_0805_Side" (id 2) (at 156.21 97.79 0)
       (effects (font (size 1.27 1.27)) hide)
     )
@@
     )
     (path "/a7b0874a-33e3-4c73-a4a5-d025cfbcc21c"
-      (reference "D1") (unit 1) (value "LED") (footprint "LED_SMD:LED_0805_2012Metric")
+      (reference "D1") (unit 1) (value "LED") (footprint "LED_SMD:LED_0805_Side")
     )
     (path "/3748fe33-2fdd-4f69-8b78-54539af3cf7b"
-      (reference "D2") (unit 1) (value "LED") (footprint "LED_SMD:LED_0805_2012Metric")
+      (reference "D2") (unit 1) (value "LED") (footprint "LED_SMD:LED_0805_Side")
     )
     (path "/0f6af24a-7399-494d-ba7b-7da6dab06934"
-      (reference "D3") (unit 1) (value "LED") (footprint "LED_SMD:LED_0805_2012Metric")
+      (reference "D3") (unit 1) (value "LED") (footprint "LED_SMD:LED_0805_Side")
     )
     (path "/b71a3c3d-b910-49dc-8b51-51df976812c9"
-      (reference "D4") (unit 1) (value "LED") (footprint "LED_SMD:LED_0805_2012Metric")
+      (reference "D4") (unit 1) (value "LED") (footprint "LED_SMD:LED_0805_Side")
     )
     (path "/3bac745c-8c11-4a7a-94f7-ef0ea55807fc"
-      (reference "D5") (unit 1) (value "LED") (footprint "LED_SMD:LED_0805_2012Metric")
+      (reference "D5") (unit 1) (value "LED") (footprint "LED_SMD:LED_0805_Side")
     )
     (path "/693813b2-df0e-40f4-b59f-935115912580"

Commit message: Okay, one more tweak because of some supply issues with the battery case
Parts:
- BT2: footprint Battery:BatteryHolder_Keystone_3034_1x20mm -> Battery:BatteryHolder_Keystone_1060_1x2032; LCSC C964834 -> C70377
Changed lines of the file:
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@@
       (effects (font (size 1.27 1.27)) (justify left))
     )
-    (property "Footprint" "Battery:BatteryHolder_Keystone_3034_1x20mm" (id 2) (at 172.72 92.456 90)
+    (property "Footprint" "Battery:BatteryHolder_Keystone_1060_1x2032" (id 2) (at 172.72 92.456 90)
       (effects (font (size 1.27 1.27)) hide)
     )
@@
       (effects (font (size 1.27 1.27)) hide)
     )
-    (property "LCSC" "C964834" (id 4) (at 172.72 93.98 0)
+    (property "LCSC" "C70377" (id 4) (at 172.72 93.98 0)
       (effects (font (size 1.27 1.27)) hide)
     )
@@
   (symbol_instances
     (path "/487a0111-ea79-4599-b0a6-5bca494e314e"
-      (reference "BT2") (unit 1) (value "Battery_Cell") (footprint "Battery:BatteryHolder_Keystone_3034_1x20mm")
+      (reference "BT2") (unit 1) (value "Battery_Cell") (footprint "Battery:BatteryHolder_Keystone_1060_1x2032")
     )
     (path "/a7b0874a-33e3-4c73-a4a5-d025cfbcc21c"
